File: KiCad/WifiFlex-connector.kicad_pcb (KiCad board)
At the start: 2 copper layers, 28.8 x 10.5 mm, 1 part, among them J1 Conn_01x20_Pin

Commit message: logo proposal
-logo and silk labels added in 8.0RC1
Other:
- board text added: "2024"
- board text added: "bitbuilt.net"
- board text added: "supertazon & yveltal"
